File: KiCad/Main Board/Electronic Target.kicad_sch (KiCad schematic)
At the start: 119 parts, among them J1 0475890001, J10 JST_PH_1x2, J11 Header 4x2, J2 640456-6, J3 EBWA-04-B, J4 BHR-12-UVA, J5 JST_PH_1x2, J6 JST_PH_1x2, J7 JST_PH_1x2, J8 JST_PH_1x2, J9 JST_PH_1x2, Q1 DWN1019UVT-7, Q2 DMN1019UVT-7, U1 FT230XS-U, U10 ESP32-WROOM-23D_DEV, U11 LM75AIMX_NOPB, U2 LM339, U3 MCP6004, U4 MCP6004, U5 ICE40UP5K-SG48ITR, U6 PDSE1-S5-D6-M-TR, U7 AP2127N-3.3, U8 AP2127N-1.2, U9 AP2127N-3.3, X1 ASFL1-64.000MHZ-EC-T

Commit message: esp 32 staging
Parts:
- added J?: B3B-PH-K-S, symbol Connector:Conn_01x03_Male
- added U?: W25Q32JVSS, Package_SO:SOIC-8_5.23x5.23mm_P1.27mm, symbol Memory_Flash:W25Q32JVSS
Connections:
- net +3V3: now also X1.1 (EN), U?.8 (VCC)
- net BD_REV: no longer U10.23 (A13_IO15)
- net CTS-U: now also U10.12 (A16_IO14); no longer U10.5 (A6_IO34)
- net GND: now also J?.3 (Pin_3), U?.4 (GND)
- net LED_PWM: now also U10.10 (A19_IO26); no longer U10.3 (A0_IO36)
- net MIC_EAST: now also U10.5 (A6_IO34)
- net MIC_NORTH: now also U10.4 (A3_IO39)
- net MIC_SOUTH: now also U10.6 (A7_IO35)
- net MIC_WEST: now also U10.7 (A4_IO32)
- net RTS-U: now also U10.11 (A17_IO27); no longer U10.4 (A3_IO39)
- net SCL: now also U?.1 (~CS)
- net SPARE_1: now also U10.8 (A5_IO33); no longer U10.6 (A7_IO35)
- net SPARE_2: now also U10.9 (A18_IO25); no longer U10.7 (A4_IO32)
- net SPISS_SDA: now also U?.6 (CLK)
- net VCC: now also J?.1 (Pin_1)
- net V_FB: now also U10.3 (A0_IO36)
- net miso: now also U?.5 (DI(IO0))
- net mosi: now also U?.2 (DO(IO1))
- net pixels: now also J?.2 (Pin_2)
- net at J11.2 (Pin_2): now also U5.36 (IOT_48b); no longer U10.8 (A5_IO33)
- net at J11.4 (Pin_4): now also U5.43 (IOT_49a); no longer U10.9 (A18_IO25)
- net at J11.6 (Pin_6): now also U5.38 (IOT_50b); no longer U10.10 (A19_IO26)
- net at J11.8 (Pin_8): now also U5.42 (IOT_51a); no longer U10.11 (A17_IO27)
- net QUIET: no longer names the net of U10.18 (CMD_IO_11)
- net QUIET: no longer X1.1 (EN)
- no-connect marks 26 -> 22
Other:
- note added: "External LEDs"
- moved on the sheet: J11, R37, R38
