File: KiCad/Main Board/Electronic Target.kicad_sch (KiCad schematic)
At the start: 121 parts, among them J1 0475890001, J10 JST_PH_1x2, J11 Header 4x2, J2 640456-6, J3 EBWA-04-B, J4 BHR-12-UVA, J5 JST_PH_1x2, J6 JST_PH_1x2, J7 JST_PH_1x2, J8 JST_PH_1x2, J9 JST_PH_1x2, Q1 DWN1019UVT-7, Q2 DMN1019UVT-7, U1 FT230XS-U, U10 ESP32-WROOM-23D_DEV, U11 LM75AIMX_NOPB, U2 LM339, U3 MCP6004, U4 MCP6004, U5 ICE40UP5K-SG48ITR, U6 PDSE1-S5-D6-M-TR, U7 AP2127N-3.3, U8 AP2127N-1.2, U9 AP2127N-3.3, X1 ASFL1-64.000MHZ-EC-T

Commit message: initial laypout
Parts:
- removed J1: 0475890001, symbol Connector_Generic:Conn_01x05
- removed J3: EBWA-04-B, symbol Connector_Generic:Conn_01x04
- removed Q1: DWN1019UVT-7, symbol Device:Q_NMOS_DGS
- removed Q2: DMN1019UVT-7, symbol Device:Q_NMOS_DGS
- removed R7: 2k2, symbol Device:R
- removed U6: PDSE1-S5-D6-M-TR, NMA0505SC:SIP600W50P254L1950H1000Q5, symbol Electronic-Target-rescue:NMA0505SC-NMA0505SC-Electronic-Target-rescue-Electroni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
- removed U?: W25Q32JVSS, Package_SO:SOIC-8_5.23x5.23mm_P1.27mm, symbol Memory_Flash:W25Q32JVSS
- added 1, 2, E2, F1, F2, F3, F4, F5, F6, GND, RGB1, RGB2, RGB3, V1: TP, Connector_PinHeader_2.54mm:PinHeader_1x01_P2.54mm_Vertical, symbol Connector_Generic:Conn_01x01
- added ADD LED: B3B-PH-K-S, Connector_JST:JST_EH_B3B-EH-A_1x03_P2.50mm_Vertical, symbol Connector:Conn_01x03_Male
- added C10: 4.7uF, Capacitor_SMD:C_0603_1608Metric, symbol UPduino_v3.0:Device_C
- added C11, C31, C6: 0.1uF, Capacitor_SMD:C_0603_1608Metric, symbol Device:C
- added C32: 10uF, Capacitor_SMD:C_0603_1608Metric, symbol Device:CP
- added D5: B5819WS-TP, Diode_SMD:D_SOD-323, symbol Device:D_Schottky
- added J3: PH5442264, TerminalBlock_Phoenix:TerminalBlock_Phoenix_PT-1,5-4-3.5-H_1x04_P3.50mm_Horizontal, symbol Connector:Screw_Terminal_01x04
- added J4: USB_B_Mini, Connector_USB:USB_Mini-B_Lumberg_2486_01_Horizontal, symbol Connector:USB_B_Mini
- added Q1, Q2: DMN1010UVT, Package_TO_SOT_SMD:TSOT-23-6, symbol DMN1019UVT:DMN1010UVT
- added U1: NMA0505SC, Converter_DCDC:Converter_DCDC_muRata_NMAxxxxSC_THT, symbol Regulator_Switching:NMA0505SC
- AUX: renamed from J2; value 640456-6 -> TE640456-6; footprint (none) -> Connector_PinHeader_2.54mm:PinHeader_1x06_P2.54mm_Vertical
- C1: renamed from C9; footprint Resistor_SMD:R_1206_3216Metric -> Capacitor_SMD:C_0603_1608Metric
- C12: renamed from C17; value 0u1 -> 0.1uF; footprint Resistor_SMD:R_0805_2012Metric -> Capacitor_SMD:C_0603_1608Metric
- C13: renamed from C11; value 4.7u -> 4.7uF
- C14: renamed from C10; value 0.1u -> 0.1uF
- C15: renamed from C22; value 0u1 -> 0.1uF; footprint Resistor_SMD:R_0805_2012Metric -> Capacitor_SMD:C_0603_1608Metric
- C16: renamed from C20; value 0u1 -> 0.1uF; footprint Resistor_SMD:R_0805_2012Metric -> Capacitor_SMD:C_0603_1608Metric
- C17: renamed from C33; value 4.7u -> 4.7uF
- C18: value 4.7u -> 4.7uF
- C19: renamed from C15; value 4.7u -> 4.7uF
- C2: renamed from C7; footprint Resistor_SMD:R_1206_3216Metric -> Capacitor_SMD:C_0603_1608Metric
- C20: renamed from C24; value 0u1 -> 0.1uF; footprint Resistor_SMD:R_0805_2012Metric -> Capacitor_SMD:C_0603_1608Metric
- C21: renamed from C32; footprint Resistor_SMD:R_1210_3225Metric -> Capacitor_SMD:C_0603_1608Metric
- C22: renamed from C39; value 680P -> 200P; footprint (none) -> Capacitor_SMD:C_0603_1608Metric
- C23: renamed from C36; value 0u1 -> 0.1uF; footprint Resistor_SMD:R_0805_2012Metric -> Capacitor_SMD:C_0603_1608Metric
- C24: renamed from C8; value 4.7u -> 4.7uF; footprint (none) -> Capacitor_SMD:C_0603_1608Metric
- C25: renamed from C12; footprint Resistor_SMD:R_1210_3225Metric -> Capacitor_SMD:C_0603_1608Metric
- C26: renamed from C13; value 0u1 -> 0.1uF; footprint Resistor_SMD:R_0805_2012Metric -> Capacitor_SMD:C_0603_1608Metric
- C27: renamed from C23; value 4.7u -> 4.7uF
- C28: renamed from C37; footprint Resistor_SMD:R_1210_3225Metric -> Capacitor_SMD:C_0603_1608Metric
- C29: renamed from C41; value 680P -> 200P; footprint (none) -> Capacitor_SMD:C_0603_1608Metric
- C3: renamed from C14; value 0u1 -> 0.1uF; footprint Resistor_SMD:R_0805_2012Metric -> Capacitor_SMD:C_0603_1608Metric
- C30: renamed from C40; value 680P -> 200P; footprint (none) -> Capacitor_SMD:C_0603_1608Metric
- C33: renamed from C19; value 0u1 -> 0.1uF; footprint Resistor_SMD:R_0805_2012Metric -> Capacitor_SMD:C_0603_1608Metric
- C34: renamed from 0u1F1; footprint (none) -> Capacitor_SMD:C_0603_1608Metric
- C35: renamed from C4; footprint (none) -> Capacitor_SMD:C_0603_1608Metric
- C36: renamed from C2; footprint (none) -> Capacitor_SMD:C_0603_1608Metric
- C37: renamed from C1; value 0u1F -> 0.1uF; footprint (none) -> Capacitor_SMD:C_0603_1608Metric
- C38: renamed from C21; value 0.1u -> 0.1uF
- C39: renamed from C27; footprint (none) -> Capacitor_SMD:C_0603_1608Metric
- C4: renamed from C38; value 680P -> 200P; footprint (none) -> Capacitor_SMD:C_0603_1608Metric
- C40: renamed from C26; footprint (none) -> Capacitor_SMD:C_0603_1608Metric
- C41: renamed from C25; footprint (none) -> Capacitor_SMD:C_0603_1608Metric
- C42: renamed from C29; footprint (none) -> Capacitor_SMD:C_0603_1608Metric
- C43: renamed from C30; footprint (none) -> Capacitor_SMD:C_0603_1608Metric
- C44: renamed from C28; footprint (none) -> Capacitor_SMD:C_0603_1608Metric
- C45: renamed from C16; value 0u1 -> 0.1uF; footprint Resistor_SMD:R_0805_2012Metric -> Capacitor_SMD:C_0603_1608Metric
- C46: renamed from C5; value 4u7F -> 4.7uF; footprint (none) -> Capacitor_SMD:C_0603_1608Metric
- C47: renamed from C31; value 4.7u -> 4.7uF
- C5: renamed from C35; value 680P -> 200P; footprint (none) -> Capacitor_SMD:C_0603_1608Metric
- C7: renamed from C6; footprint Resistor_SMD:R_1206_3216Metric -> Capacitor_SMD:C_0603_1608Metric
- C8: renamed from C3; value 0u1F -> 0.1uF; footprint (none) -> Capacitor_SMD:C_0603_1608Metric
- C9: renamed from C34; value 680P -> 200P; footprint (none) -> Capacitor_SMD:C_0603_1608Metric
- EXT LED: renamed from J?; footprint (none) -> Connector_JST:JST_EH_B3B-EH-A_1x03_P2.50mm_Vertical
- J1: renamed from J4; footprint (none) -> Connector_PinHeader_2.54mm:PinHeader_2x06_P2.54mm_Vertical
- R1: renamed from R2; footprint (none) -> Resistor_SMD:R_0603_1608Metric
- R10: renamed from R16; value 10k -> 10K; footprint (none) -> Resistor_SMD:R_0603_1608Metric
- R11: renamed from R23; value 10k -> 10K; footprint (none) -> Resistor_SMD:R_0603_1608Metric
- R12: renamed from R8; value 2k2 -> 3.3K; footprint (none) -> Resistor_SMD:R_0603_1608Metric
- R13: value 10k -> 10K; footprint (none) -> Resistor_SMD:R_0603_1608Metric
- R14: renamed from R27; value 10k -> 10K; footprint (none) -> Resistor_SMD:R_0603_1608Metric
- R15: footprint (none) -> Resistor_SMD:R_0603_1608Metric
- R16: renamed from R14; value 10k -> 10K; footprint (none) -> Resistor_SMD:R_0603_1608Metric
- R17: renamed from R24; value 10k -> 10K; footprint (none) -> Resistor_SMD:R_0603_1608Metric
- R18: renamed from R25; value 10k -> 10K; footprint (none) -> Resistor_SMD:R_0603_1608Metric
- R19: renamed from R32; value 10K -> 3.3K; footprint (none) -> Resistor_SMD:R_0603_1608Metric
- R2: renamed from R10; footprint Resistor_SMD:R_0805_2012Metric -> Resistor_SMD:R_0603_1608Metric
- R20: renamed from R9; value 2k2 -> 3.3K; footprint (none) -> Resistor_SMD:R_0603_1608Metric
- R22: renamed from R28; value 10k -> 10K; footprint (none) -> Resistor_SMD:R_0603_1608Metric
- R23: renamed from R26; value 10k -> 10K; footprint (none) -> Resistor_SMD:R_0603_1608Metric
- R24: renamed from R34; value 10K -> 3.3K; footprint (none) -> Resistor_SMD:R_0603_1608Metric
- R25: renamed from R33; value 10K -> 3.3K; footprint (none) -> Resistor_SMD:R_0603_1608Metric
- R26: renamed from R36; value 4K7 -> 4.7K; footprint Resistor_SMD:R_0805_2012Metric -> Resistor_SMD:R_0603_1608Metric
- R27: renamed from R3; value 4k7 -> 4.7K; footprint (none) -> Resistor_SMD:R_0603_1608Metric
- R28: renamed from R5; footprint (none) -> Resistor_SMD:R_0603_1608Metric
- R29: renamed from R6; footprint (none) -> Resistor_SMD:R_0603_1608Metric
- R3: renamed from R11; footprint Resistor_SMD:R_0805_2012Metric -> Resistor_SMD:R_0603_1608Metric
- R30: renamed from R35; value 4K7 -> 4.7K; footprint Resistor_SMD:R_0805_2012Metric -> Resistor_SMD:R_0603_1608Metric
- R31: renamed from R4; value 10K0 -> 10K; footprint (none) -> Resistor_SMD:R_0603_1608Metric
- R32: renamed from R19; value 2k2 -> 2.2K; footprint (none) -> Resistor_SMD:R_0603_1608Metric
- R33: renamed from R17; value 2k2 -> 2.2K; footprint (none) -> Resistor_SMD:R_0603_1608Metric
- R34: renamed from R18; value 2k2 -> 2.2K; footprint (none) -> Resistor_SMD:R_0603_1608Metric
- R35: renamed from R20; value 2k2 -> 2.2K; footprint (none) -> Resistor_SMD:R_0603_1608Metric
- R36: renamed from R22; value 2k2 -> 2.2K; footprint (none) -> Resistor_SMD:R_0603_1608Metric
- R37: renamed from R21; value 2k2 -> 2.2K; footprint (none) -> Resistor_SMD:R_0603_1608Metric
- R4: renamed from R1; footprint (none) -> Resistor_SMD:R_0603_1608Metric
- R5: renamed from R31; value 10K -> 3.3K; footprint (none) -> Resistor_SMD:R_0603_1608Metric
- R6: renamed from R30; value 10K -> 3.3K; footprint (none) -> Resistor_SMD:R_0603_1608Metric
- R7: renamed from R29; value 10K -> 3.3K; footprint (none) -> Resistor_SMD:R_0603_1608Metric
- R8: renamed from R38; footprint (none) -> Resistor_SMD:R_0603_1608Metric
- R9: renamed from R37; footprint (none) -> Resistor_SMD:R_0603_1608Metric
- RV1: value 10k0 -> 10K; footprint Digikey Pot:23BR10KLFTR -> Potentiometer_SMD:Potentiometer_Bourns_3314S_Horizontal
- U11: renamed from U1; footprint SSOP16 -> Package_SO:SSOP-16_3.9x4.9mm_P0.635mm
- U2: footprint (none) -> Package_SO:SOIC-14_3.9x8.7mm_P1.27mm
- U6: renamed from U3; footprint (none) -> Package_SO:SOIC-14_3.9x8.7mm_P1.27mm
- U8: renamed from U4; footprint (none) -> Package_SO:SOIC-14_3.9x8.7mm_P1.27mm
- U9: renamed from U10; footprint ESP32-DevKitC -> jml:ESP32-DEVKIT
- renumbered V-1 to -1, D4 to D1, D1 to D4, V3 to GND, J11 to J2, J5 to M1, J6 to M2, J7 to M3, J8 to M4, J9 to M5, J10 to M6, R12 to R21, U11 to U10, U8 to U3, U5 to U4, U7 to U5, U9 to U7, V4 to V2, V1 to V3, V2 to VCC
Connections:
- net PAPER* is gone; now on net PAPER: U9.33 (IO21)
- net +1V2: now also C11.1
- net +3.3VA: now also R2.1, RV1.1, 2.1 (Pin_1), C32.1, C6.1
- net +3V3: now also 1.1 (Pin_1), C31.1; no longer C20.1, C21.1, U9.1 (VDD33)
- net GND: now also ADD LED.3 (Pin_3), C10.2, C11.2, C31.2, C32.2, C6.2, GND.1 (Pin_1), J3.4 (Pin_4), J4.4 (ID), J4.5 (GND), J4.6 (Shield), Q1.4 (S), Q2.4 (S), U1.2 (VIN-), U1.5 (0V), V1.1 (Pin_1)
- net LED_PWM: now also Q1.3 (G)
- net PAPER: now also Q2.3 (G)
- net VCC: now also R27.1, ADD LED.1 (Pin_1), C10.1, D5.1 (K), U1.1 (VIN+); no longer R2.1, RV1.1
- net V_FB: no longer U9.3 (A0_IO36)
- net at -1.1 (Pin_1), C2.2, J1.11 (Pin_11)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: now also U1.4 (VOUT-)
- net at C1.1: now also U1.6 (VOUT+)
- net at AUX.4 (Pin_4): now also Q2.1 (D)
- net at C35.1, R29.2: now also J4.2 (D-)
- net at C36.1, R28.2: now also J4.3 (D+)
- net at C24.1, R13.2, U6.3 (+): now also R12.2
- net at U4.32 (IOT_43a): now also F2.1 (Pin_1)
- net at U4.34 (IOT_44b): now also F1.1 (Pin_1)
- net at U4.37 (IOT_45a_G1): now also F3.1 (Pin_1)
- net at U4.39 (RGB0): now also RGB3.1 (Pin_1)
- net at U4.40 (RGB1): now also RGB1.1 (Pin_1)
- net at U4.41 (RGB2): now also RGB2.1 (Pin_1)
- net at U4.18 (IOB_31b): now also F5.1 (Pin_1)
- net at U4.19 (IOB_29b): now also F6.1 (Pin_1)
- net at D1.2 (DOUT): now also ADD LED.2 (Pin_2)
- net miso: no longer names the net of U9.31 (IO19)
- net miso: now also E2.1 (Pin_1); no longer U4.14 (IOB_32a_SPI_SO)
- new net: J3.1 (Pin_1), Q1.1 (D)
- new net: J3.2 (Pin_2), J3.3 (Pin_3)
- new net: D5.2 (A), J4.1 (VBUS)
- new net: F4.1 (Pin_1), U4.14 (IOB_32a_SPI_SO)
- new net +3.3VP: C20.1, C21.1, U9.1 (VDD33)
- new net V_REFERENCE: U9.3 (A0_IO36)
- no-connect marks 22 -> 13
Other:
- note added: "Extended LEDs"
- moved on the sheet: C1, C23, C28, U7

Commit message: board updates for development board
Parts:
- removed F4, F5, F6: TP, Connector_PinHeader_2.54mm:PinHeader_1x01_P2.54mm_Vertical, symbol Connector_Generic:Conn_01x01
- removed R1, R4: 0R, Resistor_SMD:R_0603_1608Metric, symbol Device:R
- added F456, J10, J11, J12, J5, J8, J9: J1x3, Connector_PinSocket_2.54mm:PinSocket_1x03_P2.54mm_Vertical, symbol Connector:Conn_01x03_Male
- added H2: MountingHole, MountingHole:MountingHole_3.7mm, symbol Mechanical:MountingHole
- added J6: J2x3, Connector_PinHeader_2.54mm:PinHeader_2x03_P2.54mm_Vertical, symbol Connector_Generic:Conn_02x03_Odd_Even
- ADD LED1: renamed from ADD LED
- EXT LED1: renamed from EXT LED
- renumbered AUX to AUX1, GND to GND1, GND to GND2, VCC to VCC1, 2 to va33, 1 to vd33
Connections:
- net +3.3VA: now also J5.3 (Pin_3)
- net FACE_SENSOR: now also J12.1 (Pin_1)
- net GND: now also J6.2 (Pin_2), J6.5 (Pin_5)
- net MIC_EAST: now also J9.1 (Pin_1)
- net MIC_NORTH: now also J8.1 (Pin_1)
- net MIC_SOUTH: now also J10.1 (Pin_1)
- net MIC_WEST: now also J11.1 (Pin_1)
- net SD0+: now also J8.2 (Pin_2); no longer R11.1, U8.1
- net SD1+: now also J9.2 (Pin_2); no longer R17.1, U6.7
- net SD2+: now also J10.2 (Pin_2); no longer R18.1, U6.8
- net SD3+: now also J11.2 (Pin_2); no longer R23.1, U8.14
- net SD4+: now also J12.2 (Pin_2); no longer R14.1, U8.7
- net VCC: now also J5.1 (Pin_1)
- net v_bias: now also J6.6 (Pin_6)
- net M-5V: now reaches -1.1 (Pin_1), C2.2, U1.4 (VOUT-)
- net M-5V: now also J6.1 (Pin_1); no longer J1.11 (Pin_11), J1.9 (Pin_9)
- net vs+: now reaches J1.1 (Pin_1), J1.3 (Pin_3)
- net vs+: now also J5.2 (Pin_2)
- net vsb: now reaches J1.5 (Pin_5), J1.7 (Pin_7)
- net vsb: now also J6.4 (Pin_4)
- net at U4.18 (IOB_31b): now also F456.2 (Pin_2)
- net at U4.19 (IOB_29b): now also F456.3 (Pin_3)
- net at U4.14 (IOB_32a_SPI_SO): now also F456.1 (Pin_1)
- new net: J8.3 (Pin_3), R11.1, U8.1
- new net: J11.3 (Pin_3), R23.1, U8.14
- new net: J12.3 (Pin_3), R14.1, U8.7
- new net: J9.3 (Pin_3), R17.1, U6.7
- new net: J10.3 (Pin_3), R18.1, U6.8
- new net vs-: J1.11 (Pin_11), J1.9 (Pin_9), J6.3 (Pin_3)
Other:
- note added: "Jumpers to select sensor voltages, -5,0,5 or 0,1.3,3.3"
- note added: "compatable sensor board inputs and comparitors."
- note removed: "backwards compatable sensor board inputs and comparitors."
- moved on the sheet: C39, C40, C41, C42, C43, C44, M1, M2, M3, M4, M5, M6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

Commit message: stage for next merge
Parts:
- R3: value 1K5 -> 2.2k
Connections:
- net at AUX1.4 (Pin_4), Q2.1 (D): now also Q2.2 (D), Q2.5 (D), Q2.6 (D)
- net at J3.1 (Pin_1), Q1.1 (D): now also Q1.2 (D), Q1.5 (D), Q1.6 (D)
Changed lines of the file:
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@@
   (junction (at 414.02 36.83) (diameter 1.016) (color 0 0 0 0))
   (junction (at 414.02 39.37) (diameter 1.016) (color 0 0 0 0))
-  (no_connect (at 378.46 135.89))
-  (no_connect (at 378.46 105.41))
-  (no_connect (at 378.46 102.87))
   (no_connect (at 85.09 187.96))
-  (no_connect (at 358.14 39.37))
-  (no_connect (at 85.09 185.42))
-  (no_connect (at 340.36 135.89))
   (no_connect (at 85.09 190.5))
+  (no_connect (at 85.09 185.42))
   (no_connect (at 340.36 138.43))
-  (no_connect (at 378.46 140.97))
-  (no_connect (at 378.46 138.43))
+  (no_connect (at 378.46 102.87))
+  (no_connect (at 378.46 105.41))
   (no_connect (at 337.82 97.79))
   (no_connect (at 340.36 133.35))
+  (no_connect (at 378.46 135.89))
+  (no_connect (at 378.46 140.97))
+  (no_connect (at 340.36 135.89))
+  (no_connect (at 358.14 39.37))
+  (no_connect (at 378.46 138.43))
   (wire (pts (xy 13.97 193.04) (xy 13.97 194.31))
     (stroke (width 0) (type solid) (color 0 0 0 0))
@@
       (effects (font (size 1.27 1.27)) (justify left))
     )
-    (property "Value" "1K5" (id 1) (at 116.078 53.213 0)
+    (property "Value" "2.2k" (id 1) (at 116.078 53.213 0)
       (effects (font (size 1.27 1.27)) (justify left))
     )
@@
     )
   )
-  (symbol (lib_id "Connector_Generic:Conn_02x04_Odd_Even") (at 110.49 97.79 0) (unit 1)
-    (in_bom yes) (on_board yes)
-    (property "Reference" "J2" (id 0) (at 111.76 98.6282 0))
-    (property "Value" "Header 4x2" (id 1) (at 111.76 92.0496 0))
-    (property "Footprint" "Connector_PinHeader_2.54mm:PinHeader_2x04_P2.54mm_Vertical" (id 2) (at 110.49 97.79 0)
-      (effects (font (size 1.27 1.27)) hide)
-    )
-    (property "Datasheet" "~" (id 3) (at 110.49 97.79 0)
-      (effects (font (size 1.27 1.27)) hide)
-    )
-  )
   (symbol (lib_id "DMN1019UVT:DMN1010UVT") (at 24.13 118.11 0) (mirror y) (unit 1)
     (in_bom yes) (on_board yes)
@@
     )
   )
-  (symbol (lib_id "DMN1019UVT:DMN1010UVT") (at 27.94 128.27 0) (mirror y) (unit 1)
+  (symbol (lib_name "DMN1019UVT:DMN1010UVT_1") (lib_id "DMN1019UVT:DMN1010UVT") (at 27.94 128.27 0) (mirror y) (unit 1)
     (in_bom yes) (on_board yes)
     (property "Reference" "Q2" (id 0) (at 31.75 124.46 0)
@@
     )
   )
+  (symbol (lib_id "Connector_Generic:Conn_02x04_Odd_Even") (at 110.49 97.79 0) (unit 1)
+    (in_bom yes) (on_board yes)
+    (property "Reference" "J2" (id 0) (at 111.76 98.6282 0))
+    (property "Value" "Header 4x2" (id 1) (at 111.76 92.0496 0))
+    (property "Footprint" "Connector_PinHeader_2.54mm:PinHeader_2x04_P2.54mm_Vertical" (id 2) (at 110.49 97.79 0)
+      (effects (font (size 1.27 1.27)) hide)
+    )
+    (property "Datasheet" "~" (id 3) (at 110.49 97.79 0)
+      (effects (font (size 1.27 1.27)) hide)
+    )
+  )
   (symbol (lib_id "Regulator_Linear:AP2127N-3.3") (at 180.34 214.63 0) (unit 1)
     (in_bom yes) (on_board yes)
@@
     )
     (path "/00000000-0000-0000-0000-00005ef511bf"
-      (reference "R3") (unit 1) (value "1K5") (footprint "Resistor_SMD:R_0603_1608Metric")
+      (reference "R3") (unit 1) (value "2.2k") (footprint "Resistor_SMD:R_0603_1608Metric")
     )
     (path "/964d8d33-3dff-4ef5-ab71-0a2a99efef40"
